File: msp430_remote.kicad_pcb (KiCad board)
At the start: 2 copper layers, 15 parts, among them K1 CONN_3, P1 CONN_4, P2 CONN_5, P3 CONN_4X2, P4 CONN_4, U1 MSP430G2553IPW20

Commit message: tudo_feito
Parts:
- moved D1 57.8 mm to (252.7, 179.1), turned to 180 degrees
Connections:
- U1 pad 3: N-0000013 -> (no net)
- U1 pad 4: N-0000014 -> (no net)
Routing:
- net GND: track 47.6 -> 97.7 mm, vias 0 -> 6
- net +3.3V: track 98.8 -> 110.4 mm
- net /IRQ: track 29.2 -> 34.0 mm
- net N-0000025: track 0.00 -> 3.15 mm
- net /B1: track 27.9 -> 29.0 mm
- added copper zone on F.Cu, net GND
